File: eagle/FDL-2_electronics/power.brd (EAGLE design)
At the start: 37.8 x 25.4 mm, 6 parts, among them X1 JST-XH-02-PIN-ROUND-PAD, X2 JST-XH-02-PIN-ROUND-PAD

Commit message: some changes
Parts:
- removed SV3: (no value), con-lstb:MA04-1
- added SV1: (no value), con-lstb:MA05-1
- added U$1: MP2315, mylib:MP2315
- moved SV4 37.4 mm to (39.4, 7.62), turned to 90 degrees
- moved X1 24.2 mm to (8.89, 14.0)
- moved X2 24.2 mm to (8.89, 5.08)
- moved SV5 22.5 mm to (10.2, 27.9), turned to 270 degrees
- moved U$2 7.41 mm to (24.1, 10.2), turned to 0 degrees
Connections:
- new net N$5: SV5.3, U$1.P$2, U$2.P$3, X1.1
- new net N$6: SV1.5, U$2.P$13
- net N$14: now also SV1.2, U$2.P$16; no longer SV3.2, U$2.P$9
- net N$21: now also SV1.3, U$2.P$15; no longer SV3.3, U$2.P$10
- net N$22: now also SV1.4, U$2.P$14; no longer SV3.4, U$2.P$11
- net N$24: now also U$2.P$9; no longer U$2.P$16
- net N$25: now also SV1.1; no longer SV3.1
- net N$3: now also U$1.P$1, U$2.P$1; no longer SV5.3, U$2.P$3, X1.1
- net N$4: now also U$1.P$3; no longer U$2.P$1
Routing:
- net N$5: track 0.00 -> 33.1 mm
- net N$4: track 11.2 -> 27.0 mm
- net N$3: track 18.6 -> 3.81 mm
- net N$6: track 0.00 -> 9.94 mm
- net N$25: track 17.4 -> 23.2 mm
- net N$22: track 7.40 -> 9.94 mm
- net N$14: track 7.40 -> 9.94 mm
- net N$21: track 7.40 -> 9.94 mm
- net N$24: track 7.62 -> 9.94 mm
- net N$1: track 12.5 -> 11.7 mm
Other:
- board size 37.8 x 25.4 mm -> 46.7 x 34.3 mm
- board text added: "46,4 x 34"

Commit message: some update
Parts:
- removed SV5: (no value), con-lstb:MA03-1
- removed U$1: MP2315, mylib:MP2315
- added POWER_A: MA03-1, con-lstb:MA03-1
- X1: value JST-XH-02-PIN-ROUND-PAD -> Power
- X2: value JST-XH-02-PIN-ROUND-PAD -> Motor
- renumbered SV1 to PUSHER_A, SV4 to ESC
Connections:
- removed net N$3: U$1.P$1, U$2.P$1
- net N$28: now also POWER_A.2; no longer SV5.2
- net N$4: now also POWER_A.3, U$2.P$1; no longer SV5.1, U$1.P$3
- net N$5: now also POWER_A.1; no longer SV5.3, U$1.P$2
Routing:
- net N$4: track 27.0 -> 13.8 mm
- net N$5: track 33.1 -> 19.9 mm
- net N$3: track 3.81 -> 0.00 mm
- net N$28: track 20.1 -> 22.4 mm
Changed lines of the file:
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@@
 </autorouter>
 <elements>
-<element name="SV4" library="con-lstb" library_urn="urn:adsk.eagle:library:162" package="MA03-2" package3d_urn="urn:adsk.eagle:package:8334/1" value="" x="39.37" y="7.62" rot="R90">
+<element name="ESC" library="con-lstb" library_urn="urn:adsk.eagle:library:162" package="MA03-2" package3d_urn="urn:adsk.eagle:package:8334/1" value="" x="39.37" y="7.62" rot="R90">
 <attribute name="MF" value="" x="39.37" y="7.62" size="1.778" layer="27" rot="R90" display="off"/>
 <attribute name="MPN" value="" x="39.37" y="7.62" size="1.778" layer="27" rot="R90" display="off"/>
@@
 <attribute name="OC_NEWARK" value="unknown" x="39.37" y="7.62" size="1.778" layer="27" rot="R90" display="off"/>
 </element>
-<element name="SV5" library="con-lstb" library_urn="urn:adsk.eagle:library:162" package="MA03-1" package3d_urn="urn:adsk.eagle:package:8339/1" value="" x="10.16" y="27.94" rot="R270">
-<attribute name="MF" value="" x="10.16" y="27.94" size="1.778" layer="27" rot="R270" display="off"/>
-<attribute name="MPN" value="" x="10.16" y="27.94" size="1.778" layer="27" rot="R270" display="off"/>
-<attribute name="OC_FARNELL" value="unknown" x="10.16" y="27.94" size="1.778" layer="27" rot="R270" display="off"/>
-<attribute name="OC_NEWARK" value="unknown" x="10.16" y="27.94" size="1.778" layer="27" rot="R270" display="off"/>
-</element>
 <element name="U$2" library="mylib" package="TB6612FNG" value="TB6612FNG" x="24.13" y="10.16"/>
-<element name="X1" library="Rembrandt Electronics - JST XH Connectors v1-0" package="JST-XH-02-PACKAGE-ROUND-PAD" value="JST-XH-02-PIN-ROUND-PAD" x="8.89" y="13.97" rot="R90"/>
-<element name="X2" library="Rembrandt Electronics - JST XH Connectors v1-0" package="JST-XH-02-PACKAGE-ROUND-PAD" value="JST-XH-02-PIN-ROUND-PAD" x="8.89" y="5.08" rot="R90"/>
-<element name="U$1" library="mylib" package="MP2315" value="MP2315" x="66.04" y="27.94"/>
-<element name="SV1" library="con-lstb" package="MA05-1" package3d_urn="urn:adsk.eagle:package:8332/1" value="" x="40.64" y="20.32" rot="R270">
+<element name="X1" library="Rembrandt Electronics - JST XH Connectors v1-0" package="JST-XH-02-PACKAGE-ROUND-PAD" value="Power" x="8.89" y="13.97" rot="R90"/>
+<element name="X2" library="Rembrandt Electronics - JST XH Connectors v1-0" package="JST-XH-02-PACKAGE-ROUND-PAD" value="Motor" x="8.89" y="5.08" rot="R90"/>
+<element name="PUSHER_A" library="con-lstb" package="MA05-1" package3d_urn="urn:adsk.eagle:package:8332/1" value="" x="40.64" y="20.32" rot="R270">
 <attribute name="MF" value="" x="40.64" y="20.32" size="1.778" layer="27" rot="R270" display="off"/>
 <attribute name="MPN" value="" x="40.64" y="20.32" size="1.778" layer="27" rot="R270" display="off"/>
@@
 <attribute name="OC_NEWARK" value="unknown" x="40.64" y="20.32" size="1.778" layer="27" rot="R270" display="off"/>
 </element>
+<element name="POWER_A" library="con-lstb" package="MA03-1" value="MA03-1" x="7.62" y="21.59"/>
 </elements>
 <signals>
@@
 <wire x1="31.75" y1="20.32" x2="34.29" y2="20.32" width="0.8128" layer="16"/>
 <wire x1="34.29" y1="20.32" x2="36.83" y2="22.86" width="0.8128" layer="16"/>
-<contactref element="SV1" pad="2"/>
+<contactref element="PUSHER_A" pad="2"/>
 <wire x1="36.83" y1="22.86" x2="40.64" y2="22.86" width="0.8128" layer="16"/>
 </signal>
@@
 <wire x1="31.75" y1="17.78" x2="34.29" y2="17.78" width="0.8128" layer="16"/>
 <wire x1="34.29" y1="17.78" x2="36.83" y2="20.32" width="0.8128" layer="16"/>
-<contactref element="SV1" pad="3"/>
+<contactref element="PUSHER_A" pad="3"/>
 <wire x1="36.83" y1="20.32" x2="40.64" y2="20.32" width="0.8128" layer="16"/>
 </signal>
@@
 <wire x1="31.75" y1="15.24" x2="34.29" y2="15.24" width="0.8128" layer="16"/>
 <wire x1="34.29" y1="15.24" x2="36.83" y2="17.78" width="0.8128" layer="16"/>
-<contactref element="SV1" pad="4"/>
+<contactref element="PUSHER_A" pad="4"/>
 <wire x1="36.83" y1="17.78" x2="40.64" y2="17.78" width="0.8128" layer="16"/>
 </signal>
 <signal name="N$24">
 <contactref element="U$2" pad="P$9"/>
-<contactref element="SV4" pad="2"/>
-<contactref element="SV4" pad="1"/>
+<contactref element="ESC" pad="2"/>
+<contactref element="ESC" pad="1"/>
 <wire x1="31.75" y1="2.54" x2="34.29" y2="2.54" width="0.8128" layer="16"/>
 <wire x1="34.29" y1="2.54" x2="36.83" y2="5.08" width="0.8128" layer="16"/>
@@
 </signal>
 <signal name="N$25">
-<contactref element="SV4" pad="6"/>
-<contactref element="SV4" pad="5"/>
+<contactref element="ESC" pad="6"/>
+<contactref element="ESC" pad="5"/>
 <wire x1="38.1" y1="10.16" x2="40.64" y2="10.16" width="0.8128" layer="16"/>
 <wire x1="40.64" y1="10.16" x2="41.91" y2="10.16" width="0.8128" layer="16"/>
@@
 <wire x1="43.18" y1="25.4" x2="44.45" y2="24.13" width="0.8128" layer="16"/>
 <wire x1="41.91" y1="10.16" x2="44.45" y2="12.7" width="0.8128" layer="16"/>
-<contactref element="SV1" pad="1"/>
+<contactref element="PUSHER_A" pad="1"/>
 <wire x1="40.64" y1="25.4" x2="43.18" y2="25.4" width="0.8128" layer="16"/>
 </signal>
 <signal name="N$28">
-<contactref element="SV5" pad="2"/>
 <contactref element="U$2" pad="P$2"/>
-<wire x1="10.16" y1="27.94" x2="8.89" y2="27.94" width="0.8128" layer="16"/>
-<wire x1="8.89" y1="27.94" x2="7.62" y2="26.67" width="0.8128" layer="16"/>
-<wire x1="7.62" y1="26.67" x2="7.62" y2="19.05" width="0.8128" layer="16"/>
-<wire x1="7.62" y1="19.05" x2="8.89" y2="17.78" width="0.8128" layer="16"/>
-<wire x1="8.89" y1="17.78" x2="16.51" y2="17.78" width="0.8128" layer="16"/>
+<contactref element="POWER_A" pad="2"/>
+<wire x1="7.62" y1="21.59" x2="10.16" y2="24.13" width="0.8128" layer="16"/>
+<wire x1="10.16" y1="24.13" x2="19.05" y2="24.13" width="0.8128" layer="16"/>
+<wire x1="19.05" y1="24.13" x2="20.32" y2="22.86" width="0.8128" layer="16"/>
+<wire x1="20.32" y1="22.86" x2="20.32" y2="19.05" width="0.8128" layer="16"/>
+<wire x1="20.32" y1="19.05" x2="19.05" y2="17.78" width="0.8128" layer="16"/>
+<wire x1="19.05" y1="17.78" x2="16.51" y2="17.78" width="0.8128" layer="16"/>
 </signal>
 <signal name="N$1">
@@
 </signal>
 <signal name="N$5">
-<contactref element="SV5" pad="3"/>
 <contactref element="U$2" pad="P$3"/>
 <contactref element="X1" pad="1"/>
-<contactref element="U$1" pad="P$2"/>
-<wire x1="10.16" y1="25.4" x2="12.7" y2="25.4" width="0.8128" layer="16"/>
-<wire x1="12.7" y1="25.4" x2="13.97" y2="26.67" width="0.8128" layer="16"/>
-<wire x1="13.97" y1="26.67" x2="16.51" y2="26.67" width="0.8128" layer="16"/>
-<wire x1="16.51" y1="26.67" x2="19.05" y2="26.67" width="0.8128" layer="16"/>
-<wire x1="19.05" y1="26.67" x2="20.32" y2="25.4" width="0.8128" layer="16"/>
-<wire x1="20.32" y1="25.4" x2="20.32" y2="16.51" width="0.8128" layer="16"/>
-<wire x1="20.32" y1="16.51" x2="19.05" y2="15.24" width="0.8128" layer="16"/>
-<wire x1="19.05" y1="15.24" x2="16.51" y2="15.24" width="0.8128" layer="16"/>
-<wire x1="16.51" y1="15.24" x2="13.97" y2="15.24" width="0.8128" layer="16"/>
-<wire x1="13.97" y1="15.24" x2="11.43" y2="12.7" width="0.8128" layer="16"/>
-<wire x1="11.43" y1="12.7" x2="8.89" y2="12.7" width="0.8128" layer="16"/>
+<wire x1="8.89" y1="12.7" x2="10.16" y2="12.7" width="0.8128" layer="16"/>
+<wire x1="10.16" y1="12.7" x2="12.7" y2="15.24" width="0.8128" layer="16"/>
+<wire x1="12.7" y1="15.24" x2="16.51" y2="15.24" width="0.8128" layer="16"/>
+<contactref element="POWER_A" pad="1"/>
+<wire x1="8.89" y1="12.7" x2="7.62" y2="12.7" width="0.8128" layer="16"/>
+<wire x1="7.62" y1="12.7" x2="5.08" y2="15.24" width="0.8128" layer="16"/>
+<wire x1="5.08" y1="15.24" x2="5.08" y2="21.59" width="0.8128" layer="16"/>
 </signal>
 <signal name="N$4">
 <contactref element="X1" pad="2"/>
-<contactref element="U$1" pad="P$3"/>
-<contactref element="SV5" pad="1"/>
-<wire x1="10.16" y1="30.48" x2="12.7" y2="30.48" width="0.8128" layer="16"/>
-<wire x1="12.7" y1="30.48" x2="13.97" y2="29.21" width="0.8128" layer="16"/>
-<wire x1="13.97" y1="29.21" x2="16.51" y2="29.21" width="0.8128" layer="16"/>
-<wire x1="8.89" y1="15.24" x2="7.62" y2="15.24" width="0.8128" layer="16"/>
-<wire x1="7.62" y1="15.24" x2="6.35" y2="16.51" width="0.8128" layer="16"/>
-<wire x1="6.35" y1="16.51" x2="6.35" y2="29.21" width="0.8128" layer="16"/>
-<wire x1="6.35" y1="29.21" x2="7.62" y2="30.48" width="0.8128" layer="16"/>
-<wire x1="7.62" y1="30.48" x2="10.16" y2="30.48" width="0.8128" layer="16"/>
-</signal>
-<signal name="N$3">
-<contactref element="U$1" pad="P$1"/>
 <contactref element="U$2" pad="P$1"/>
-<wire x1="16.51" y1="24.13" x2="16.51" y2="20.32" width="0.8128" layer="16"/>
+<contactref element="POWER_A" pad="3"/>
+<wire x1="10.16" y1="21.59" x2="11.43" y2="20.32" width="0.8128" layer="16"/>
+<wire x1="11.43" y1="20.32" x2="16.51" y2="20.32" width="0.8128" layer="16"/>
+<wire x1="11.43" y1="20.32" x2="11.43" y2="16.51" width="0.8128" layer="16"/>
+<wire x1="11.43" y1="16.51" x2="10.16" y2="15.24" width="0.8128" layer="16"/>
+<wire x1="10.16" y1="15.24" x2="8.89" y2="15.24" width="0.8128" layer="16"/>
 </signal>
 <signal name="N$6">
-<contactref element="SV1" pad="5"/>
+<contactref element="PUSHER_A" pad="5"/>
 <contactref element="U$2" pad="P$13"/>
 <wire x1="31.75" y1="12.7" x2="34.29" y2="12.7" width="0.8128" layer="16"/>

Commit message: some further work - mainly on pusher
Parts:
- added C1: (no value), resistor:TT5D7
- moved ESC 1.80 mm to (40.6, 6.35)
- moved PUSHER_A 1.80 mm to (39.4, 19.1)
Connections:
- net N$28: now also C1.+
- net N$5: now also C1.-
Routing:
- net N$5: track 19.9 -> 36.7 mm
- net N$9: track 9.94 -> 8.15 mm
- net N$8: track 9.94 -> 8.15 mm
- net N$6: track 9.94 -> 8.15 mm
- net N$3: track 9.94 -> 8.15 mm
- net N$25: track 23.2 -> 21.4 mm
- net N$28: track 22.4 -> 23.2 mm
- net N$24: track 9.94 -> 10.7 mm
Other:
- board size 46.7 x 34.3 mm -> 46.4 x 34 mm
- board text added: "AI1"
- board text added: "AI2"
- board text added: "AO1"
- board text added: "AO2"
- board text added: "GND"
- board text added: "PWM"
- board text added: "STBY"
- board text added: "VCC"
- board text added: "VM"
