File: eagle/FDL-2_electronics/power.sch (EAGLE design)
At the start: 6 parts, among them X1 JST-XH-02-PIN-ROUND-PAD, X2 JST-XH-02-PIN-ROUND-PAD

Commit message: some changes
Parts:
- removed SV3: (no value), con-lstb:MA04-1
- added SV1: (no value), con-lstb:MA05-1
- added U$1: MP2315, mylib:MP2315
Connections:
- new net N$5: SV5.3, U$1.GND, U$2.GND@1, X1-1.S
- new net N$6: SV1.5, U$2.STBY
- net N$14: now also SV1.2; no longer SV3.2
- net N$21: now also SV1.3; no longer SV3.3
- net N$22: now also SV1.4; no longer SV3.4
- net N$25: now also SV1.1; no longer SV3.1
- net N$3: now also U$1.VO+, U$2.VM; no longer SV5.3, U$2.GND@1, X1-1.S
- net N$4: now also U$1.IN+; no longer U$2.VM
Other:
- moved on the sheet: X1-1, X1-2
Changed lines of the file:
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@@
 <parts>
 <part name="U$2" library="mylib" deviceset="TB6612FNG" device=""/>
-<part name="SV3" library="con-lstb" library_urn="urn:adsk.eagle:library:162" deviceset="MA04-1" device="" package3d_urn="urn:adsk.eagle:package:8337/1"/>
 <part name="SV4" library="con-lstb" library_urn="urn:adsk.eagle:library:162" deviceset="MA03-2" device="" package3d_urn="urn:adsk.eagle:package:8334/1"/>
 <part name="SV5" library="con-lstb" library_urn="urn:adsk.eagle:library:162" deviceset="MA03-1" device="" package3d_urn="urn:adsk.eagle:package:8339/1"/>
 <part name="X1" library="Rembrandt Electronics - JST XH Connectors v1-0" deviceset="JST-XH-02-PIN" device="-ROUND-PAD"/>
 <part name="X2" library="Rembrandt Electronics - JST XH Connectors v1-0" deviceset="JST-XH-02-PIN" device="-ROUND-PAD"/>
+<part name="U$1" library="mylib" deviceset="MP2315" device=""/>
+<part name="SV1" library="con-lstb" deviceset="MA05-1" device="" package3d_urn="urn:adsk.eagle:package:8332/1"/>
 </parts>
 <sheets>
@@
 </plain>
 <instances>
-<instance part="U$2" gate="G$1" x="25.4" y="45.72"/>
-<instance part="SV3" gate="1" x="68.58" y="63.5" rot="R180"/>
+<instance part="U$2" gate="G$1" x="30.48" y="45.72"/>
 <instance part="SV4" gate="1" x="66.04" y="40.64"/>
 <instance part="SV5" gate="G$1" x="-10.16" y="63.5" rot="MR180"/>
-<instance part="X1" gate="-2" x="7.62" y="78.74"/>
-<instance part="X1" gate="-1" x="7.62" y="81.28"/>
+<instance part="X1" gate="-2" x="27.94" y="83.82"/>
+<instance part="X1" gate="-1" x="27.94" y="86.36"/>
 <instance part="X2" gate="-2" x="7.62" y="33.02"/>
 <instance part="X2" gate="-1" x="7.62" y="35.56"/>
+<instance part="U$1" gate="G$1" x="-15.24" y="86.36"/>
+<instance part="SV1" gate="G$1" x="68.58" y="63.5" rot="R180"/>
 </instances>
 <busses>
@@
 <net name="N$14" class="0">
 <segment>
-<pinref part="SV3" gate="1" pin="2"/>
 <pinref part="U$2" gate="G$1" pin="PWMA"/>
-<wire x1="60.96" y1="66.04" x2="38.1" y2="66.04" width="0.1524" layer="91"/>
+<wire x1="60.96" y1="66.04" x2="43.18" y2="66.04" width="0.1524" layer="91"/>
+<pinref part="SV1" gate="G$1" pin="2"/>
 </segment>
 </net>
 <net name="N$21" class="0">
 <segment>
-<pinref part="SV3" gate="1" pin="3"/>
 <pinref part="U$2" gate="G$1" pin="AI2"/>
-<wire x1="60.96" y1="63.5" x2="38.1" y2="63.5" width="0.1524" layer="91"/>
+<wire x1="60.96" y1="63.5" x2="43.18" y2="63.5" width="0.1524" layer="91"/>
+<pinref part="SV1" gate="G$1" pin="3"/>
 </segment>
 </net>
 <net name="N$22" class="0">
 <segment>
-<pinref part="SV3" gate="1" pin="4"/>
 <pinref part="U$2" gate="G$1" pin="AI1"/>
-<wire x1="60.96" y1="60.96" x2="38.1" y2="60.96" width="0.1524" layer="91"/>
+<wire x1="60.96" y1="60.96" x2="43.18" y2="60.96" width="0.1524" layer="91"/>
+<pinref part="SV1" gate="G$1" pin="4"/>
 </segment>
 </net>
@@
 <segment>
 <pinref part="U$2" gate="G$1" pin="GND@3"/>
-<wire x1="38.1" y1="48.26" x2="50.8" y2="48.26" width="0.1524" layer="91"/>
+<wire x1="43.18" y1="48.26" x2="50.8" y2="48.26" width="0.1524" layer="91"/>
 <wire x1="50.8" y1="48.26" x2="50.8" y2="38.1" width="0.1524" layer="91"/>
 <pinref part="SV4" gate="1" pin="2"/>
@@
 <net name="N$25" class="0">
 <segment>
-<pinref part="SV3" gate="1" pin="1"/>
 <wire x1="60.96" y1="68.58" x2="55.88" y2="68.58" width="0.1524" layer="91"/>
 <wire x1="55.88" y1="68.58" x2="55.88" y2="50.8" width="0.1524" layer="91"/>
@@
 <wire x1="76.2" y1="50.8" x2="55.88" y2="50.8" width="0.1524" layer="91"/>
 <junction x="55.88" y="50.8"/>
+<pinref part="SV1" gate="G$1" pin="1"/>
 </segment>
 </net>
@@
 <pinref part="SV5" gate="G$1" pin="2"/>
 <pinref part="U$2" gate="G$1" pin="VCC"/>
-<wire x1="-2.54" y1="63.5" x2="10.16" y2="63.5" width="0.1524" layer="91"/>
+<wire x1="-2.54" y1="63.5" x2="15.24" y2="63.5" width="0.1524" layer="91"/>
 </segment>
 </net>
@@
 <segment>
 <pinref part="U$2" gate="G$1" pin="A01"/>
-<wire x1="10.16" y1="58.42" x2="0" y2="58.42" width="0.1524" layer="91"/>
+<wire x1="15.24" y1="58.42" x2="0" y2="58.42" width="0.1524" layer="91"/>
 <wire x1="0" y1="58.42" x2="0" y2="33.02" width="0.1524" layer="91"/>
 <pinref part="X2" gate="-2" pin="S"/>
@@
 <segment>
 <pinref part="U$2" gate="G$1" pin="A02"/>
-<wire x1="10.16" y1="55.88" x2="2.54" y2="55.88" width="0.1524" layer="91"/>
+<wire x1="15.24" y1="55.88" x2="2.54" y2="55.88" width="0.1524" layer="91"/>
 <pinref part="X2" gate="-1" pin="S"/>
 <wire x1="2.54" y1="55.88" x2="2.54" y2="35.56" width="0.1524" layer="91"/>
@@
 </segment>
 </net>
-<net name="N$3" class="0">
+<net name="N$5" class="0">
 <segment>
+<pinref part="U$2" gate="G$1" pin="GND@1"/>
 <pinref part="SV5" gate="G$1" pin="3"/>
-<pinref part="U$2" gate="G$1" pin="GND@1"/>
-<wire x1="-2.54" y1="60.96" x2="0" y2="60.96" width="0.1524" layer="91"/>
+<wire x1="-2.54" y1="60.96" x2="5.08" y2="60.96" width="0.1524" layer="91"/>
 <pinref part="X1" gate="-1" pin="S"/>
-<wire x1="0" y1="60.96" x2="10.16" y2="60.96" width="0.1524" layer="91"/>
-<wire x1="5.08" y1="81.28" x2="0" y2="81.28" width="0.1524" layer="91"/>
-<wire x1="0" y1="81.28" x2="0" y2="60.96" width="0.1524" layer="91"/>
-<junction x="0" y="60.96"/>
+<pinref part="U$1" gate="G$1" pin="GND"/>
+<wire x1="5.08" y1="60.96" x2="15.24" y2="60.96" width="0.1524" layer="91"/>
+<wire x1="25.4" y1="86.36" x2="5.08" y2="86.36" width="0.1524" layer="91"/>
+<wire x1="5.08" y1="86.36" x2="0" y2="86.36" width="0.1524" layer="91"/>
+<wire x1="5.08" y1="60.96" x2="5.08" y2="86.36" width="0.1524" layer="91"/>
+<junction x="5.08" y="60.96"/>
+<junction x="5.08" y="86.36"/>
 </segment>
 </net>
@@
 <segment>
 <pinref part="X1" gate="-2" pin="S"/>
-<wire x1="5.08" y1="78.74" x2="2.54" y2="78.74" width="0.1524" layer="91"/>
+<pinref part="U$1" gate="G$1" pin="IN+"/>
+<wire x1="25.4" y1="83.82" x2="2.54" y2="83.82" width="0.1524" layer="91"/>
 <pinref part="SV5" gate="G$1" pin="1"/>
-<pinref part="U$2" gate="G$1" pin="VM"/>
+<wire x1="2.54" y1="83.82" x2="0" y2="83.82" width="0.1524" layer="91"/>
 <wire x1="-2.54" y1="66.04" x2="2.54" y2="66.04" width="0.1524" layer="91"/>
-<wire x1="2.54" y1="66.04" x2="10.16" y2="66.04" width="0.1524" layer="91"/>
-<wire x1="2.54" y1="78.74" x2="2.54" y2="66.04" width="0.1524" layer="91"/>
-<junction x="2.54" y="66.04"/>
+<wire x1="2.54" y1="83.82" x2="2.54" y2="66.04" width="0.1524" layer="91"/>
+<junction x="2.54" y="83.82"/>
 </segment>
 </net>
+<net name="N$3" class="0">
+<segment>
+<pinref part="U$1" gate="G$1" pin="VO+"/>
+<wire x1="0" y1="88.9" x2="7.62" y2="88.9" width="0.1524" layer="91"/>
+<wire x1="7.62" y1="88.9" x2="7.62" y2="66.04" width="0.1524" layer="91"/>
+<pinref part="U$2" gate="G$1" pin="VM"/>
+<wire x1="7.62" y1="66.04" x2="15.24" y2="66.04" width="0.1524" layer="91"/>
+</segment>
+</net>
+<net name="N$6" class="0">
+<segment>
+<pinref part="SV1" gate="G$1" pin="5"/>
+<pinref part="U$2" gate="G$1" pin="STBY"/>
+<wire x1="60.96" y1="58.42" x2="43.18" y2="58.42" width="0.1524" layer="91"/>
+</segment>
+</net>

Commit message: some update
Parts:
- removed U$1: MP2315, mylib:MP2315
- POWER_A: value (none) -> MA03-1
- X1: value JST-XH-02-PIN-ROUND-PAD -> Power
- X2: value JST-XH-02-PIN-ROUND-PAD -> Motor
- renumbered SV1 to PUSHER_A, SV4 to ESC, SV5 to POWER_A
Connections:
- removed net N$3: U$1.VO+, U$2.VM
- net N$4: now also POWER_A.3, U$2.VM; no longer POWER_A.1, U$1.IN+
- net N$5: now also POWER_A.1; no longer POWER_A.3, U$1.GND
Other:
- moved on the sheet: X1-1, X1-2, X2-1, X2-2

Commit message: some further work - mainly on pusher
Parts:
- added C1: (no value), resistor:CPOL-EUTT5D7
Connections:
- net N$28: now also C1.+
- net N$5: now also C1.-
