File: eagle/FDL-2_electronics/main.brd (EAGLE design)
At the start: 47.4 x 34.2 mm, 10 parts

Commit message: some fixes
Routing:
- net N$15: track 30.5 -> 27.1 mm
- net N$16: track 30.7 -> 29.9 mm
Changed lines of the file:
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@@
 <contactref element="S1" pad="SW-"/>
 <contactref element="B1" pad="19"/>
-<wire x1="27.705" y1="17.669575" x2="28.450425" y2="18.415" width="0.6096" layer="16"/>
-<wire x1="28.450425" y1="18.415" x2="29.21" y2="18.415" width="0.6096" layer="16"/>
+<wire x1="27.705" y1="17.669575" x2="29.085425" y2="17.78" width="0.6096" layer="16"/>
+<wire x1="29.085425" y1="17.78" x2="29.21" y2="18.415" width="0.6096" layer="16"/>
 <wire x1="29.21" y1="18.415" x2="35.433" y2="24.638" width="0.6096" layer="16"/>
 <wire x1="35.433" y1="24.638" x2="36.068" y2="24.638" width="0.6096" layer="16"/>
@@
 <contactref element="B1" pad="A4"/>
 <contactref element="SV2" pad="4"/>
-<wire x1="24.8475" y1="19.098325" x2="24.799175" y2="19.05" width="0.6096" layer="16"/>
-<wire x1="24.799175" y1="19.05" x2="22.86" y2="19.05" width="0.6096" layer="16"/>
-<wire x1="19.05" y1="31.75" x2="16.51" y2="32.385" width="0.6096" layer="16"/>
-<wire x1="16.51" y1="32.385" x2="8.255" y2="32.385" width="0.6096" layer="16"/>
-<wire x1="8.255" y1="32.385" x2="9.525" y2="31.75" width="0.6096" layer="16"/>
+<wire x1="24.8475" y1="19.098325" x2="23.543325" y2="19.098325" width="0.6096" layer="16"/>
+<wire x1="23.543325" y1="19.098325" x2="23.495" y2="19.05" width="0.6096" layer="16"/>
+<wire x1="23.495" y1="19.05" x2="18.415" y2="24.13" width="0.6096" layer="16"/>
+<wire x1="17.145" y1="32.385" x2="10.16" y2="32.385" width="0.6096" layer="16"/>
+<wire x1="10.16" y1="32.385" x2="9.525" y2="31.75" width="0.6096" layer="16"/>
 <wire x1="9.525" y1="31.75" x2="9.525" y2="29.845" width="0.6096" layer="16"/>
-<wire x1="22.86" y1="19.05" x2="19.05" y2="22.86" width="0.6096" layer="16"/>
-<wire x1="19.05" y1="22.86" x2="19.05" y2="31.75" width="0.6096" layer="16"/>
+<wire x1="18.415" y1="24.13" x2="18.415" y2="31.115" width="0.6096" layer="16"/>
+<wire x1="18.415" y1="31.115" x2="17.145" y2="32.385" width="0.6096" layer="16"/>
 </signal>
 <signal name="N$16">
@@
 <wire x1="20.2692" y1="24.8158" x2="20.2692" y2="32.2550125" width="0.6096" layer="16"/>
 <wire x1="20.2692" y1="32.2550125" x2="18.8692125" y2="33.655" width="0.6096" layer="16"/>
-<wire x1="7.62" y1="33.655" x2="6.985" y2="33.02" width="0.6096" layer="16"/>
-<wire x1="6.985" y1="33.02" x2="6.985" y2="29.845" width="0.6096" layer="16"/>
-<wire x1="18.8692125" y1="33.655" x2="7.62" y2="33.655" width="0.6096" layer="16"/>
+<wire x1="8.89" y1="33.655" x2="6.985" y2="31.75" width="0.6096" layer="16"/>
+<wire x1="6.985" y1="31.75" x2="6.985" y2="29.845" width="0.6096" layer="16"/>
+<wire x1="18.8692125" y1="33.655" x2="8.89" y2="33.655" width="0.6096" layer="16"/>
 </signal>
 <signal name="N$18">
 <contactref element="B1" pad="15"/>
 <contactref element="SV1" pad="3"/>
-<wire x1="29.845" y1="7.62" x2="27.815425" y2="7.62" width="0.6096" layer="16"/>
+<wire x1="29.21" y1="7.62" x2="27.815425" y2="7.62" width="0.6096" layer="16"/>
 <wire x1="27.815425" y1="7.62" x2="27.705" y2="7.509575" width="0.6096" layer="16"/>
-<wire x1="31.8008" y1="5.6642" x2="29.845" y2="7.62" width="0.6096" layer="16"/>
+<wire x1="31.1658" y1="5.6642" x2="29.21" y2="7.62" width="0.6096" layer="16"/>
 <wire x1="41.275" y1="2.54" x2="41.275" y2="3.81" width="0.6096" layer="16"/>
 <wire x1="41.275" y1="3.81" x2="39.4208" y2="5.6642" width="0.6096" layer="16"/>
-<wire x1="39.4208" y1="5.6642" x2="31.8008" y2="5.6642" width="0.6096" layer="16"/>
+<wire x1="39.4208" y1="5.6642" x2="31.1658" y2="5.6642" width="0.6096" layer="16"/>
 </signal>
 <signal name="N$17">
@@
 <wire x1="38.735" y1="2.54" x2="38.735" y2="3.81" width="0.6096" layer="16"/>
 <wire x1="38.735" y1="3.81" x2="38.1" y2="4.445" width="0.6096" layer="16"/>
-<wire x1="38.1" y1="4.445" x2="31.115" y2="4.445" width="0.6096" layer="16"/>
-<wire x1="31.115" y1="4.445" x2="30.48" y2="5.08" width="0.6096" layer="16"/>
-<wire x1="30.48" y1="5.08" x2="27.815425" y2="5.08" width="0.6096" layer="16"/>
+<wire x1="38.1" y1="4.445" x2="29.845" y2="4.445" width="0.6096" layer="16"/>
+<wire x1="29.845" y1="4.445" x2="29.21" y2="5.08" width="0.6096" layer="16"/>
+<wire x1="29.21" y1="5.08" x2="27.815425" y2="5.08" width="0.6096" layer="16"/>
 <wire x1="27.815425" y1="5.08" x2="27.705" y2="4.969575" width="0.6096" layer="16"/>
 </signal>
@@
 <wire x1="19.374225" y1="34.8742" x2="7.1149875" y2="34.8742" width="0.6096" layer="16"/>
 <wire x1="7.1149875" y1="34.8742" x2="5.2607875" y2="33.02" width="0.6096" layer="16"/>
-<wire x1="2.54" y1="33.02" x2="1.905" y2="32.385" width="0.6096" layer="16"/>
-<wire x1="1.905" y1="32.385" x2="1.905" y2="29.845" width="0.6096" layer="16"/>
-<wire x1="5.2607875" y1="33.02" x2="2.54" y2="33.02" width="0.6096" layer="16"/>
+<wire x1="3.175" y1="33.02" x2="1.905" y2="31.75" width="0.6096" layer="16"/>
+<wire x1="1.905" y1="31.75" x2="1.905" y2="29.845" width="0.6096" layer="16"/>
+<wire x1="5.2607875" y1="33.02" x2="3.175" y2="33.02" width="0.6096" layer="16"/>
 <wire x1="20.1392125" y1="34.1092125" x2="20.32" y2="34.29" width="0.6096" layer="16"/>
 <wire x1="40.64" y1="34.29" x2="41.275" y2="33.655" width="0.6096" layer="16"/>

Commit message: some changes
Parts:
- removed SV1: (no value), con-lstb:MA04-1
- added SV3: (no value), con-lstb:MA05-1
Connections:
- net N$17: now also SV3.P$4; no longer SV1.4
- net N$18: now also SV3.P$3; no longer SV1.3
- net N$19: now also SV3.P$2; no longer SV1.2
- net N$2: now also SV3.P$5
- net N$20: now also SV3.P$1; no longer SV1.1
Routing:
- net N$2: track 0.00 -> 33.6 mm
- net N$19: track 12.9 -> 10.2 mm
- net N$20: track 8.54 -> 6.00 mm
- net N$18: track 16.5 -> 14.2 mm
- net N$17: track 20.0 -> 17.7 mm
Other:
- board size 47.4 x 34.2 mm -> 46.7 x 36.1 mm
Changed lines of the file:
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@@
 <board>
 <plain>
-<wire x1="0" y1="1.27" x2="47.365" y2="1.27" width="0" layer="20"/>
-<wire x1="47.365" y1="1.27" x2="47.365" y2="35.46" width="0" layer="20"/>
-<wire x1="47.365" y1="35.46" x2="0" y2="35.46" width="0" layer="20"/>
-<wire x1="0" y1="35.46" x2="0" y2="1.27" width="0" layer="20"/>
-<dimension x1="0" y1="0" x2="47.365" y2="0" x3="23.6825" y3="-3.81" textsize="1.778" layer="16"/>
-<dimension x1="0" y1="1.27" x2="0" y2="36.195" x3="-2.54" y3="18.7325" textsize="1.778" layer="1"/>
+<wire x1="0" y1="0" x2="46.73" y2="0" width="0" layer="20"/>
+<wire x1="46.73" y1="0" x2="46.73" y2="36.095" width="0" layer="20"/>
+<wire x1="46.73" y1="36.095" x2="0" y2="36.095" width="0" layer="20"/>
+<wire x1="0" y1="36.095" x2="0" y2="0" width="0" layer="20"/>
+<dimension x1="0" y1="0" x2="0" y2="36.195" x3="-3.175" y3="18.0975" textsize="1.778" layer="16"/>
+<dimension x1="0" y1="0" x2="46.73" y2="0" x3="23.365" y3="-3.81" textsize="1.778" layer="16"/>
 </plain>
 <attributes>
@@
 <element name="FIRE" library="con-lstb" package="MA03-1" value="" x="5.715" y="15.24"/>
 <element name="U$1" library="con-lstb" package="MA03-1" value="MA03-1" x="41.275" y="31.115"/>
-<element name="SV1" library="con-lstb" package="MA04-1" package3d_urn="urn:adsk.eagle:package:8337/1" value="" x="40.005" y="2.54">
-<attribute name="MF" value="" x="40.005" y="2.54" size="1.778" layer="27" display="off"/>
-<attribute name="MPN" value="" x="40.005" y="2.54" size="1.778" layer="27" display="off"/>
-<attribute name="OC_FARNELL" value="unknown" x="40.005" y="2.54" size="1.778" layer="27" display="off"/>
-<attribute name="OC_NEWARK" value="unknown" x="40.005" y="2.54" size="1.778" layer="27" display="off"/>
+<element name="SV3" library="con-lstb" package="MA05-1" package3d_urn="urn:adsk.eagle:package:8332/1" value="" x="38.735" y="2.54">
+<attribute name="MF" value="" x="38.735" y="2.54" size="1.778" layer="27" display="off"/>
+<attribute name="MPN" value="" x="38.735" y="2.54" size="1.778" layer="27" display="off"/>
+<attribute name="OC_FARNELL" value="unknown" x="38.735" y="2.54" size="1.778" layer="27" display="off"/>
+<attribute name="OC_NEWARK" value="unknown" x="38.735" y="2.54" size="1.778" layer="27" display="off"/>
 </element>
 </elements>
@@
 <signal name="N$2">
 <contactref element="B1" pad="12"/>
+<contactref element="SV3" pad="P$5"/>
+<wire x1="12.465" y1="2.429575" x2="23.605425" y2="2.429575" width="0.6096" layer="16"/>
+<wire x1="23.605425" y1="2.429575" x2="25.3492" y2="0.6858" width="0.6096" layer="16"/>
+<wire x1="43.2308" y1="0.6858" x2="43.815" y2="1.27" width="0.6096" layer="16"/>
+<wire x1="43.815" y1="1.27" x2="43.815" y2="2.54" width="0.6096" layer="16"/>
+<wire x1="25.3492" y1="0.6858" x2="43.2308" y2="0.6858" width="0.6096" layer="16"/>
 </signal>
 <signal name="N$10">
@@
 <signal name="N$18">
 <contactref element="B1" pad="15"/>
-<contactref element="SV1" pad="3"/>
-<wire x1="29.21" y1="7.62" x2="27.815425" y2="7.62" width="0.6096" layer="16"/>
-<wire x1="27.815425" y1="7.62" x2="27.705" y2="7.509575" width="0.6096" layer="16"/>
-<wire x1="31.1658" y1="5.6642" x2="29.21" y2="7.62" width="0.6096" layer="16"/>
-<wire x1="41.275" y1="2.54" x2="41.275" y2="3.81" width="0.6096" layer="16"/>
-<wire x1="41.275" y1="3.81" x2="39.4208" y2="5.6642" width="0.6096" layer="16"/>
-<wire x1="39.4208" y1="5.6642" x2="31.1658" y2="5.6642" width="0.6096" layer="16"/>
+<contactref element="SV3" pad="P$3"/>
+<wire x1="27.705" y1="7.509575" x2="29.320425" y2="7.509575" width="0.6096" layer="16"/>
+<wire x1="29.320425" y1="7.509575" x2="30.48" y2="6.35" width="0.6096" layer="16"/>
+<wire x1="30.48" y1="6.35" x2="36.83" y2="6.35" width="0.6096" layer="16"/>
+<wire x1="36.83" y1="6.35" x2="38.735" y2="4.445" width="0.6096" layer="16"/>
+<wire x1="38.735" y1="4.445" x2="38.735" y2="2.5908" width="0.6096" layer="16"/>
+<wire x1="38.735" y1="2.5908" x2="38.735" y2="2.54" width="0" layer="19" extent="16-16"/>
 </signal>
 <signal name="N$17">
 <contactref element="B1" pad="16"/>
-<contactref element="SV1" pad="4"/>
-<wire x1="43.815" y1="2.54" x2="43.815" y2="3.81" width="0.6096" layer="16"/>
-<wire x1="43.815" y1="3.81" x2="40.7416" y2="6.8834" width="0.6096" layer="16"/>
-<wire x1="40.7416" y1="6.8834" x2="32.385" y2="6.8834" width="0.6096" layer="16"/>
-<wire x1="32.385" y1="6.8834" x2="29.218825" y2="10.049575" width="0.6096" layer="16"/>
-<wire x1="29.218825" y1="10.049575" x2="27.705" y2="10.049575" width="0.6096" layer="16"/>
+<contactref element="SV3" pad="P$4"/>
+<wire x1="27.705" y1="10.049575" x2="28.5046375" y2="10.049575" width="0.6096" layer="16"/>
+<wire x1="30.9342125" y1="7.62" x2="38.1" y2="7.62" width="0.6096" layer="16"/>
+<wire x1="38.1" y1="7.62" x2="41.275" y2="4.445" width="0.6096" layer="16"/>
+<wire x1="41.275" y1="4.445" x2="41.275" y2="2.5908" width="0.6096" layer="16"/>
+<wire x1="28.5046375" y1="10.049575" x2="30.9342125" y2="7.62" width="0.6096" layer="16"/>
+<wire x1="41.275" y1="2.5908" x2="41.275" y2="2.54" width="0" layer="19" extent="16-16"/>
 </signal>
 <signal name="N$19">
 <contactref element="B1" pad="14"/>
-<contactref element="SV1" pad="2"/>
-<wire x1="38.735" y1="2.54" x2="38.735" y2="3.81" width="0.6096" layer="16"/>
-<wire x1="38.735" y1="3.81" x2="38.1" y2="4.445" width="0.6096" layer="16"/>
-<wire x1="38.1" y1="4.445" x2="29.845" y2="4.445" width="0.6096" layer="16"/>
-<wire x1="29.845" y1="4.445" x2="29.21" y2="5.08" width="0.6096" layer="16"/>
-<wire x1="29.21" y1="5.08" x2="27.815425" y2="5.08" width="0.6096" layer="16"/>
-<wire x1="27.815425" y1="5.08" x2="27.705" y2="4.969575" width="0.6096" layer="16"/>
+<contactref element="SV3" pad="P$2"/>
+<wire x1="27.705" y1="4.969575" x2="35.035425" y2="4.969575" width="0.6096" layer="16"/>
+<wire x1="35.035425" y1="4.969575" x2="36.195" y2="3.81" width="0.6096" layer="16"/>
+<wire x1="36.195" y1="3.81" x2="36.195" y2="2.5908" width="0.6096" layer="16"/>
+<wire x1="36.195" y1="2.5908" x2="36.195" y2="2.54" width="0" layer="19" extent="16-16"/>
 </signal>
 <signal name="N$20">
 <contactref element="B1" pad="13"/>
-<contactref element="SV1" pad="1"/>
-<wire x1="27.705" y1="2.429575" x2="36.084575" y2="2.429575" width="0.6096" layer="16"/>
-<wire x1="36.084575" y1="2.429575" x2="36.195" y2="2.54" width="0.6096" layer="16"/>
+<contactref element="SV3" pad="P$1"/>
+<wire x1="27.705" y1="2.429575" x2="32.909575" y2="2.429575" width="0.6096" layer="16"/>
+<wire x1="32.909575" y1="2.429575" x2="33.02" y2="2.54" width="0.6096" layer="16"/>
+<wire x1="33.02" y1="2.54" x2="33.655" y2="2.54" width="0.6096" layer="16"/>
 </signal>
 <signal name="N$23">

Commit message: update resistors
Parts:
- R1: value (none) -> 120k
- R2: value (none) -> 10k
Changed lines of the file:
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@@
 <?xml version="1.0" encoding="utf-8"?>
 <!DOCTYPE eagle SYSTEM "eagle.dtd">
-<eagle version="8.5.0">
+<eagle version="9.0.0">
 <drawing>
 <settings>
@@
 <attribute name="SF_SKU" value="COM-09117" x="38.608" y="17.653" size="1.778" layer="27" rot="R270" display="off"/>
 </element>
-<element name="R1" library="rcl" library_urn="urn:adsk.eagle:library:334" package="0204/5" package3d_urn="urn:adsk.eagle:package:23488/1" value="" x="34.925" y="29.845" rot="R270"/>
-<element name="R2" library="rcl" library_urn="urn:adsk.eagle:library:334" package="0204V" package3d_urn="urn:adsk.eagle:package:23495/1" value="" x="32.385" y="28.575" rot="R270"/>
+<element name="R1" library="rcl" library_urn="urn:adsk.eagle:library:334" package="0204/5" package3d_urn="urn:adsk.eagle:package:23488/1" value="120k" x="34.925" y="29.845" rot="R270"/>
+<element name="R2" library="rcl" library_urn="urn:adsk.eagle:library:334" package="0204V" package3d_urn="urn:adsk.eagle:package:23495/1" value="10k" x="32.385" y="28.575" rot="R270"/>
 <element name="SV2" library="con-lstb" package="MA04-1" package3d_urn="urn:adsk.eagle:package:8337/1" value="" x="5.715" y="29.845">
 <attribute name="MF" value="" x="5.715" y="29.845" size="1.778" layer="27" display="off"/>
